File: Hardware/Power_Supply.kicad_sch (KiCad schematic)
At the start: 2 parts, among them U3 RPMH5.0-1.5

Commit message: Restructure VCU schema
Parts:
- U3: now left out of the parts list
Changed lines of the file:
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@@
 		(body_style 1)
 		(exclude_from_sim no)
-		(in_bom yes)
-		(on_board yes)
+		(in_bom no)
+		(on_board no)
 		(in_pos_files yes)
 		(dnp no)

Commit message: Set footprint + excludes
Parts:
- F1: now left out of the parts list
Changed lines of the file:
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@@
 		(body_style 1)
 		(exclude_from_sim no)
-		(in_bom yes)
-		(on_board yes)
+		(in_bom no)
+		(on_board no)
 		(in_pos_files yes)
 		(dnp no)
